File: hardware/multiboard_controller/Input Connectors.kicad_sch (KiCad schematic)
At the start: 10 parts, among them J1 USB_C_Receptacle, U4 MAX38908xTD

Commit message: Add ESD protection for USB 2.0 ifaces.
Other:
- moved on the sheet: C2
Changed lines of the file:
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@@
 (kicad_sch
-	(version 20231120)
+	(version 20250114)
 	(generator "eeschema")
-	(generator_version "8.0")
+	(generator_version "9.0")
 	(paper "A4")
 	(title_block
@@
 		(date "2025-02-11")
 	)
+	(text "USB Data Pins for Fastboot"
+		(exclude_from_sim no)
+		(at 141.224 85.09 0)
+		(effects
+			(font
+				(size 1.27 1.27)
+			)
+		)
+	)
+	(text "LDO for 3V3 from USB 5V"
+		(exclude_from_sim no)
+		(at 211.074 38.862 0)
+		(effects
+			(font
+				(size 1.27 1.27)
+			)
+		)
+	)
+	(text "Plug from host (includes power)\n"
+		(exclude_from_sim no)
+		(at 99.314 44.958 0)
+		(effects
+			(font
+				(size 1.27 1.27)
+			)
+		)
+	)
+	(text_box "Enable Pin. Connect this pin to a logic signal to enable (VEN high)\nor disable (VEN low) the regulator output. Connect to BIAS to\nkeep the output enabled whenever a valid supply voltage is\npresent."
+		(exclude_from_sim no)
+		(at 185.42 101.6 0)
+		(size 31.75 21.59)
+		(margins 0.9525 0.9525 0.9525 0.9525)
+		(stroke
+			(width 0)
+			(type default)
+		)
+		(fill
+			(type none)
+		)
+		(effects
+			(font
+				(size 1.27 1.27)
+			)
+			(justify left top)
+		)
+	)
 	(junction
 		(at 241.3 86.36)
@@
 	)
 	(junction
-		(at 181.61 58.42)
+		(at 187.96 58.42)
 		(diameter 0)
 		(color 0 0 0 0)
@@
 	(wire
 		(pts
-			(xy 181.61 58.42) (xy 181.61 62.23)
-		)
-		(stroke
-			(width 0)
-			(type default)
-		)
-	)
-	(wire
-		(pts
-			(xy 181.61 58.42) (xy 200.66 58.42)
+			(xy 187.96 58.42) (xy 187.96 62.23)
+		)
+		(stroke
+			(width 0)
+			(type default)
+		)
+	)
+	(wire
+		(pts
+			(xy 187.96 58.42) (xy 200.66 58.42)
 		)
 		(stroke
@@
 	(wire
 		(pts
-			(xy 181.61 76.2) (xy 181.61 69.85)
+			(xy 187.96 76.2) (xy 187.96 69.85)
 		)
 		(stroke
@@
 	(wire
 		(pts
-			(xy 116.84 58.42) (xy 181.61 58.42)
+			(xy 116.84 58.42) (xy 187.96 58.42)
 		)
 		(stroke
@@
 			(width 0)
 			(type default)
-		)
-	)
-	(text_box "Enable Pin. Connect this pin to a logic signal to enable (VEN high)\nor disable (VEN low) the regulator output. Connect to BIAS to\nkeep the output enabled whenever a valid supply voltage is\npresent."
-		(exclude_from_sim no)
-		(at 185.42 101.6 0)
-		(size 31.75 21.59)
-		(stroke
-			(width 0)
-			(type default)
-		)
-		(fill
-			(type none)
-		)
-		(effects
-			(font
-				(size 1.27 1.27)
-			)
-			(justify left top)
-		)
-	)
-	(text "USB Data Pins for Fastboot"
-		(exclude_from_sim no)
-		(at 145.542 84.836 0)
-		(effects
-			(font
-				(size 1.27 1.27)
-			)
-		)
-	)
-	(text "LDO for 3V3 from USB 5V"
-		(exclude_from_sim no)
-		(at 211.074 38.862 0)
-		(effects
-			(font
-				(size 1.27 1.27)
-			)
-		)
-	)
-	(text "Plug from host (includes power)\n"
-		(exclude_from_sim no)
-		(at 99.314 44.958 0)
-		(effects
-			(font
-				(size 1.27 1.27)
-			)
 		)
 	)
 	(label "uC Power?"
 		(at 223.52 85.09 90)
-		(fields_autoplaced yes)
 		(effects
 			(font
@@
 	(symbol
 		(lib_id "2025-02-12_02-17-00:GRM188R60J226MEA0D")
-		(at 181.61 69.85 90)
+		(at 187.96 69.85 90)
 		(unit 1)
 		(exclude_from_sim no)
@@
 		(dnp no)
 		(property "Reference" "C2"
-			(at 175.514 65.786 0)
+			(at 181.864 65.786 0)
 			(effects
 				(font
@@
 		)
 		(property "Value" "22uF"
-			(at 177.8 62.992 0)
+			(at 184.15 62.992 0)
 			(effects
 				(font
@@
 		)
 		(property "Footprint" "G-188_MUR"
-			(at 181.61 69.85 0)
+			(at 187.96 69.85 0)
 			(effects
 				(font
@@
 		)
 		(property "Datasheet" "GRM188R60J226MEA0D"
-			(at 181.61 69.85 0)
+			(at 187.96 69.85 0)
 			(effects
 				(font
@@
 		)
 		(property "Description" ""
-			(at 181.61 69.85 0)
+			(at 187.96 69.85 0)
 			(effects
 				(font
@@
 	(symbol
 		(lib_id "power:GND")
-		(at 181.61 76.2 0)
+		(at 187.96 76.2 0)
 		(unit 1)
 		(exclude_from_sim no)
@@
 		(fields_autoplaced yes)
 		(property "Reference" "#PWR03"
-			(at 181.61 82.55 0)
+			(at 187.96 82.55 0)
 			(effects
 				(font
@@
 		)
 		(property "Value" "GND"
-			(at 181.61 81.28 0)
+			(at 187.96 81.28 0)
 			(effects
 				(font
@@
 		)
 		(property "Footprint" ""
-			(at 181.61 76.2 0)
+			(at 187.96 76.2 0)
 			(effects
 				(font
@@
 		)
 		(property "Datasheet" ""
-			(at 181.61 76.2 0)
+			(at 187.96 76.2 0)
 			(effects
 				(font
@@
 		)
 		(property "Description" "Power symbol creates a global label with name \"GND\" , ground"
-			(at 181.61 76.2 0)
-			(effects
-				(font
+			(at 187.96 76.2 0)
+			(effects
+				(font
