File: hardware/multiboard_controller/usb-switch.kicad_sch (KiCad schematic)
At the start: 1 part, among them U1 max4999etj+

Commit message: Add ESD protection for USB 2.0 ifaces.
Other:
- title: (none) -> USB Switch
